File: RPIZERO/TestPoints.kicad_sch (KiCad schematic)
At the start: 5 parts

Commit message: Clean up and resetting to do the compute modual version
Parts:
- added TP5: +5v, TestPoint:TestPoint_Pad_D1.5mm, symbol Connector:TestPoint
- added TP6: GND, TestPoint:TestPoint_Pad_D1.5mm, symbol Connector:TestPoint
Connections:
- net +5: now also TP5.1
- net GND: now also TP6.1
Changed lines of the file:
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@@
 (kicad_sch (version 20210126) (generator eeschema)
   (paper "A4")
+  (global_label "+5" (shape input) (at 106.045 114.3 270)
+    (effects (font (size 1.27 1.27)) (justify right))
+    (property "Intersheet References" "${INTERSHEET_REFS}" (id 0) (at 105.9656 119.495 90)
+      (effects (font (size 1.27 1.27)) (justify right) hide)
+    )
+  )
   (global_label "+3.3" (shape input) (at 134.62 114.3 270)
     (effects (font (size 1.27 1.27)) (justify right))
@@
       (effects (font (size 1.27 1.27)) (justify right) hide)
     )
+  )
+  (symbol (lib_id "Connector:TestPoint") (at 95.885 114.3 0) (unit 1)
+    (in_bom yes) (on_board yes)
+    (property "Reference" "TP6" (id 0) (at 97.2821 111.6976 0)
+      (effects (font (size 1.27 1.27)) (justify left))
+    )
+    (property "Value" "GND" (id 1) (at 97.2821 113.9963 0)
+      (effects (font (size 1.27 1.27)) (justify left))
+    )
+    (property "Footprint" "TestPoint:TestPoint_Pad_D1.5mm" (id 2) (at 100.965 114.3 0)
+      (effects (font (size 1.27 1.27)) hide)
+    )
+    (property "Datasheet" "~" (id 3) (at 100.965 114.3 0)
+      (effects (font (size 1.27 1.27)) hide)
+    )
+    (pin "1")
+  )
+  (symbol (lib_id "Connector:TestPoint") (at 106.045 114.3 0) (unit 1)
+    (in_bom yes) (on_board yes)
+    (property "Reference" "TP5" (id 0) (at 107.4421 111.6976 0)
+      (effects (font (size 1.27 1.27)) (justify left))
+    )
+    (property "Value" "+5v" (id 1) (at 107.4421 113.9963 0)
+      (effects (font (size 1.27 1.27)) (justify left))
+    )
+    (property "Footprint" "TestPoint:TestPoint_Pad_D1.5mm" (id 2) (at 111.125 114.3 0)
+      (effects (font (size 1.27 1.27)) hide)
+    )
+    (property "Datasheet" "~" (id 3) (at 111.125 114.3 0)
+      (effects (font (size 1.27 1.27)) hide)
+    )
+    (pin "1")
   )
   (symbol (lib_id "Connector:TestPoint") (at 123.19 114.3 0) (unit 1)
@@
       (effects (font (size 1.27 1.27)) hide)
     )
+    (pin "1")
+  )
+  (symbol (lib_id "power:GND") (at 95.885 114.3 0) (unit 1)
+    (in_bom yes) (on_board yes)
+    (property "Reference" "#PWR0108" (id 0) (at 95.885 120.65 0)
+      (effects (font (size 1.27 1.27)) hide)
+    )
+    (property "Value" "GND" (id 1) (at 95.885 118.6244 0))
+    (property "Footprint" "" (id 2) (at 95.885 114.3 0)
+      (effects (font (size 1.27 1.27)) hide)
+    )
+    (property "Datasheet" "" (id 3) (at 95.885 114.3 0)
+      (effects (font (size 1.27 1.27)) hide)
+    )
