File: RPIZERO/ps.kicad_sch (KiCad schematic)
At the start: 4 parts, among them J1 USB_B, J10 TP4056, J2 Conn_01x02

Commit message: Push before big change
Chaing the charge controll Stuffs
Parts:
- J1: footprint (none) -> Connector_USB:USB_Micro-B_Amphenol_10103594-0001LF_Horizontal
Changed lines of the file:
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@@
     (property "Reference" "J1" (id 0) (at 146.177 82.55 0))
     (property "Value" "USB_B" (id 1) (at 146.177 85.09 0))
-    (property "Footprint" "" (id 2) (at 148.59 95.25 0)
+    (property "Footprint" "Connector_USB:USB_Micro-B_Amphenol_10103594-0001LF_Horizontal" (id 2) (at 148.59 95.25 0)
       (effects (font (size 1.27 1.27)) hide)
     )
