File: RPIZERO/ti92revive.kicad_pcb (KiCad board)
At the start: 2 copper layers, 205 x 113.6 mm, 175 parts, among them J10 TP4056, J2 Conn_01x02, U1 Teensy++2.0_(Arduino)

Commit message: Clean up and resetting to do the compute modual version
Parts:
- added R1: 1.5k, Resistor_SMD:R_2010_5025Metric, B.Cu at (161.2, 95.4)
- added TP5: +5v, TestPoint:TestPoint_Pad_D1.5mm, F.Cu at (134.8, 65.4)
- added TP6: GND, TestPoint:TestPoint_Pad_D1.5mm, F.Cu at (139.6, 65.6)
Changed lines of the file:
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@@
       (net 165 "Net-(D73-Pad2)") (pinfunction "2") (pintype "passive") (zone_connect 2))
   )
+  (footprint "TestPoint:TestPoint_Pad_D1.5mm" (layer "F.Cu")
+    (at 134.8 65.448)
+    (descr "SMD pad as test Point, diameter 1.5mm")
+    (tags "test point SMD pad")
+    (property "Sheetfile" "TestPoints.kicad_sch")
+    (property "Sheetname" "TestPoints")
+    (attr exclude_from_pos_files)
+    (fp_text reference "TP5" (at 0 -1.648) (layer "F.SilkS")
+      (effects (font (size 1 1) (thickness 0.15)))
+    )
+    (fp_text value "+5v" (at 0 1.75) (layer "F.Fab")
+      (effects (font (size 1 1) (thickness 0.15)))
+    )
+    (fp_text user "${REFERENCE}" (at 0 -1.65) (layer "F.Fab")
+      (effects (font (size 1 1) (thickness 0.15)))
+    )
+    (fp_circle (center 0 0) (end 0 0.95) (layer "F.SilkS") (width 0.12) (fill none))
+    (fp_circle (center 0 0) (end 1.25 0) (layer "F.CrtYd") (width 0.05) (fill none))
+    (pad "1" smd circle (at 0 0) (locked) (size 1.5 1.5) (layers "F.Cu" "F.Mask")
+      (net 15 "+5") (pinfunction "1") (pintype "passive"))
+  )
   (footprint "18650:Kbpad" (layer "F.Cu")
     (at 67.945 83.82)
@@
       (net 163 "Net-(D71-Pad2)") (pinfunction "2") (pintype "passive") (zone_connect 2))
   )
+  (footprint "TestPoint:TestPoint_Pad_D1.5mm" (layer "F.Cu")
+    (at 139.6 65.6)
+    (descr "SMD pad as test Point, diameter 1.5mm")
+    (tags "test point SMD pad")
+    (property "Sheetfile" "TestPoints.kicad_sch")
+    (property "Sheetname" "TestPoints")
+    (attr exclude_from_pos_files)
+    (fp_text reference "TP6" (at 0 -1.648) (layer "F.SilkS")
+      (effects (font (size 1 1) (thickness 0.15)))
+    )
+    (fp_text value "GND" (at 0 1.75) (layer "F.Fab")
+      (effects (font (size 1 1) (thickness 0.15)))
+    )
+    (fp_text user "${REFERENCE}" (at 0 -1.65) (layer "F.Fab")
+      (effects (font (size 1 1) (thickness 0.15)))
+    )
+    (fp_circle (center 0 0) (end 0 0.95) (layer "F.SilkS") (width 0.12) (fill none))
+    (fp_circle (center 0 0) (end 1.25 0) (layer "F.CrtYd") (width 0.05) (fill none))
+    (pad "1" smd circle (at 0 0) (locked) (size 1.5 1.5) (layers "F.Cu" "F.Mask")
+      (net 17 "GND") (pinfunction "1") (pintype "passive"))
+  )
   (footprint "18650:Kbpad" (layer "F.Cu")
     (at 80.899 49.784)
@@
       (net 129 "Net-(D37-Pad2)") (pinfunction "2") (pintype "passive") (zone_connect 2))
   )
+  (footprint "Resistor_SMD:R_2010_5025Metric" (layer "B.Cu")
+    (at 161.2 95.4 180)
+    (descr "Resistor SMD 2010 (5025 Metric), square (rectangular) end terminal, IPC_7351 nominal, (Body size source: IPC-SM-782 page 72, https://www.pcb-3d.com/wordpress/wp-content/uploads/ipc-sm-782a_amendment_1_and_2.pdf), generated with kicad-footprint-generator")
+    (tags "resistor")
+    (property "Sheetfile" "ps.kicad_sch")
+    (property "Sheetname" "PowerSupply")
+    (attr smd)
+    (fp_text reference "R1" (at 0 2.28) (layer "B.SilkS")
+      (effects (font (size 1 1) (thickness 0.15)) (justify mirror))
+    )
+    (fp_text value "1.5k" (at 0 -2.28) (layer "B.Fab")
+      (effects (font (size 1 1) (thickness 0.15)) (justify mirror))
+    )
+    (fp_text user "${REFERENCE}" (at 0 0) (layer "B.Fab")
+      (effects (font (size 1 1) (thickness 0.15)) (justify mirror))
+    )
+    (fp_line (start -1.527064 1.36) (end 1.527064 1.36) (layer "B.SilkS") (width 0.12))
+    (fp_line (start -1.527064 -1.36) (end 1.527064 -1.36) (layer "B.SilkS") (width 0.12))
+    (fp_line (start -3.18 -1.58) (end -3.18 1.58) (layer "B.CrtYd") (width 0.05))
+    (fp_line (start 3.18 1.58) (end 3.18 -1.58) (layer "B.CrtYd") (width 0.05))
+    (fp_line (start -3.18 1.58) (end 3.18 1.58) (layer "B.CrtYd") (width 0.05))
+    (fp_line (start 3.18 -1.58) (end -3.18 -1.58) (layer "B.CrtYd") (width 0.05))
+    (fp_line (start 2.5 -1.25) (end -2.5 -1.25) (layer "B.Fab") (width 0.1))
+    (fp_line (start -2.5 -1.25) (end -2.5 1.25) (layer "B.Fab") (width 0.1))
+    (fp_line (start 2.5 1.25) (end 2.5 -1.25) (layer "B.Fab") (width 0.1))
+    (fp_line (start -2.5 1.25) (end 2.5 1.25) (layer "B.Fab") (width 0.1))
+    (pad "1" smd roundrect (at -2.3125 0 180) (locked) (size 1.225 2.65) (layers "B.Cu" "B.Paste" "B.Mask") (roundrect_rratio 0.204082)
+      (net 178 "Net-(J10-Pad2)") (pintype "passive"))
+    (pad "2" smd roundrect (at 2.3125 0 180) (locked) (size 1.225 2.65) (layers "B.Cu" "B.Paste" "B.Mask") (roundrect_rratio 0.204082)
+      (net 17 "GND") (pintype "passive"))
+    (model "${KISYS3DMOD}/Resistor_SMD.3dshapes/R_2010_5025Metric.wrl"
+      (offset (xyz 0 0 0))
+      (scale (xyz 1 1 1))
+      (rotate (xyz 0 0 0))
+    )
+  )
   (footprint "Diode_SMD:D_SOD-123" (layer "B.Cu")

Commit message: Push before big change
Chaing the charge controll Stuffs
Parts:
- added J1: USB_B, Connector_USB:USB_Micro-B_Amphenol_10103594-0001LF_Horizontal, B.Cu at (219.6, 35.0)
- moved TP1 115.2 mm to (106.8, 44.2)
- moved TP2 115.2 mm to (103.6, 44.2)
- moved TP3 115.2 mm to (97.6, 44.2)
- moved TP0 115.2 mm to (110.2, 44.2)
- moved TP4 115.2 mm to (100.7, 44.2)
Other:
- board size 205 x 113.6 mm -> 205 x 117.1 mm
Changed lines of the file:
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@@
   (net 179 "Net-(J10-Pad5)")
   (net 180 "unconnected-(J10-Pad1)")
+  (net 181 "unconnected-(J1-Pad3)")
+  (net 182 "unconnected-(J1-Pad2)")
   (footprint "18650:Kbpad" (layer "F.Cu")
     (at 204.343 100.457)
@@
   )
   (footprint "TestPoint:TestPoint_Pad_D1.5mm" (layer "B.Cu")
-    (at 222 48.4 180)
+    (at 106.830952 44.2 180)
     (descr "SMD pad as test Point, diameter 1.5mm")
     (tags "test point SMD pad")
@@
   )
   (footprint "TestPoint:TestPoint_Pad_D1.5mm" (layer "B.Cu")
-    (at 212.769048 48.4 180)
+    (at 97.6 44.2 180)
     (descr "SMD pad as test Point, diameter 1.5mm")
     (tags "test point SMD pad")
@@
   )
   (footprint "TestPoint:TestPoint_Pad_D1.5mm" (layer "B.Cu")
-    (at 218.769048 48.4 180)
+    (at 103.6 44.2 180)
     (descr "SMD pad as test Point, diameter 1.5mm")
     (tags "test point SMD pad")
@@
     )
   )
+  (footprint "Connector_USB:USB_Micro-B_Amphenol_10103594-0001LF_Horizontal" (layer "B.Cu")
+    (at 219.6 35)
+    (descr "Micro USB Type B 10103594-0001LF, http://cdn.amphenol-icc.com/media/wysiwyg/files/drawing/10103594.pdf")
+    (tags "USB USB_B USB_micro USB_OTG")
+    (property "Sheetfile" "ps.kicad_sch")
+    (property "Sheetname" "PowerSupply")
+    (attr smd)
+    (fp_text reference "J1" (at 1.925 3.365) (layer "B.SilkS")
+      (effects (font (size 1 1) (thickness 0.15)) (justify mirror))
+    )
+    (fp_text value "USB_B" (at -0.025 -4.435) (layer "B.Fab")
+      (effects (font (size 1 1) (thickness 0.15)) (justify mirror))
+    )
+    (fp_text user "PCB edge" (at -0.025 -2.235) (layer "Dwgs.User")
+      (effects (font (size 0.5 0.5) (thickness 0.075)))
+    )
+    (fp_text user "${REFERENCE}" (at -0.025 0.015) (layer "B.Fab")
+      (effects (font (size 1 1) (thickness 0.15)) (justify mirror))
+    )
+    (fp_line (start 3.825 -2.735) (end 3.825 0.065) (layer "B.SilkS") (width 0.12))
+    (fp_line (start -4.175 0.065) (end -3.875 0.065) (layer "B.SilkS") (width 0.12))
+    (fp_line (start -4.175 0.065) (end -4.175 1.615) (layer "B.SilkS") (width 0.12))
+    (fp_line (start 3.825 0.065) (end 4.125 0.065) (layer "B.SilkS") (width 0.12))
+    (fp_line (start -1.325 2.865) (end -1.725 3.315) (layer "B.SilkS") (width 0.12))
+    (fp_line (start -3.875 -2.735) (end -3.875 0.065) (layer "B.SilkS") (width 0.12))
+    (fp_line (start -1.725 3.315) (end -0.925 3.315) (layer "B.SilkS") (width 0.12))
+    (fp_line (start 4.125 0.065) (end 4.125 1.615) (layer "B.SilkS") (width 0.12))
+    (fp_line (start -0.925 3.315) (end -1.325 2.865) (layer "B.SilkS") (width 0.12))
+    (fp_line (start -4.025 -2.835) (end 3.975 -2.835) (layer "Dwgs.User") (width 0.1))
+    (fp_line (start 4.14 -3.58) (end 4.14 2.88) (layer "B.CrtYd") (width 0.05))
+    (fp_line (start -4.13 2.88) (end -4.13 -3.58) (layer "B.CrtYd") (width 0.05))
+    (fp_line (start 4.14 -3.58) (end -4.13 -3.58) (layer "B.CrtYd") (width 0.05))
+    (fp_line (start -4.13 2.88) (end 4.14 2.88) (layer "B.CrtYd") (width 0.05))
+    (fp_line (start -2.975 1.615) (end 3.725 1.615) (layer "B.Fab") (width 0.12))
+    (fp_line (start 3.725 1.615) (end 3.725 -3.335) (layer "B.Fab") (width 0.12))
+    (fp_line (start 3.725 -3.335) (end -3.775 -3.335) (layer "B.Fab") (width 0.12))
+    (fp_line (start -3.775 -3.335) (end -3.775 0.865) (layer "B.Fab") (width 0.12))
+    (fp_line (start -3.775 0.865) (end -2.975 1.615) (layer "B.Fab") (width 0.12))
+    (pad "1" smd rect (at -1.325 1.765 270) (locked) (size 1.65 0.4) (layers "B.Cu" "B.Paste" "B.Mask")
+      (net 177 "Net-(J1-Pad1)") (pinfunction "VBUS") (pintype "power_out"))
+    (pad "2" smd rect (at -0.675 1.765 270) (locked) (size 1.65 0.4) (layers "B.Cu" "B.Paste" "B.Mask")
+      (net 182 "unconnected-(J1-Pad2)") (pinfunction "D-") (pintype "bidirectional"))
+    (pad "3" smd rect (at -0.025 1.765 270) (locked) (size 1.65 0.4) (layers "B.Cu" "B.Paste" "B.Mask")
+      (net 181 "unconnected-(J1-Pad3)") (pinfunction "D+") (pintype "bidirectional"))
+    (pad "4" smd rect (at 0.625 1.765 270) (locked) (size 1.65 0.4) (layers "B.Cu" "B.Paste" "B.Mask")
+      (net 17 "GND") (pinfunction "GND") (pintype "power_out"))
+    (pad "5" smd rect (at 1.275 1.765 270) (locked) (size 1.65 0.4) (layers "B.Cu" "B.Paste" "B.Mask")
+      (net 17 "GND") (pinfunction "Shield") (pintype "passive"))
+    (pad "6" smd rect (at -2.755 -0.185) (locked) (size 1.35 2) (layers "B.Cu" "B.Paste" "B.Mask"))
+    (pad "6" smd rect (at -0.985 -1.385 270) (locked) (size 2.5 1.43) (layers "B.Cu" "B.Paste" "B.Mask"))
+    (pad "6" thru_hole oval (at 2.395 1.885 270) (locked) (size 1.5 1.1) (drill oval 1.05 0.65) (layers *.Cu *.Mask))
+    (pad "6" thru_hole oval (at -2.755 -1.115 270) (locked) (size 1.7 1.35) (drill oval 1.2 0.7) (layers *.Cu *.Mask))
+    (pad "6" smd rect (at 2.725 -0.185) (locked) (size 1.35 2) (layers "B.Cu" "B.Paste" "B.Mask"))
+    (pad "6" smd rect (at 2.975 0.565) (locked) (size 1.825 0.7) (layers "B.Cu" "B.Paste" "B.Mask"))
+    (pad "6" thru_hole oval (at 2.705 -1.115 270) (locked) (size 1.7 1.35) (drill oval 1.2 0.7) (layers *.Cu *.Mask))
+    (pad "6" thru_hole oval (at -2.445 1.885 270) (locked) (size 1.5 1.1) (drill oval 1.05 0.65) (layers *.Cu *.Mask))
+    (pad "6" smd rect (at 2.875 1.885) (locked) (size 2 1.5) (layers "B.Cu" "B.Paste" "B.Mask"))
+    (pad "6" smd rect (at 0.935 -1.385 270) (locked) (size 2.5 1.43) (layers "B.Cu" "B.Paste" "B.Mask"))
+    (pad "6" smd rect (at -2.975 0.565) (locked) (size 1.825 0.7) (layers "B.Cu" "B.Paste" "B.Mask"))
+    (pad "6" smd rect (at -2.875 1.865) (locked) (size 2 1.5) (layers "B.Cu" "B.Paste" "B.Mask"))
+    (model "${KISYS3DMOD}/Connector_USB.3dshapes/USB_Micro-B_Amphenol_10103594-0001LF_Horizontal.wrl"
+      (offset (xyz 0 0 0))
+      (scale (xyz 1 1 1))
+      (rotate (xyz 0 0 0))
+    )
+  )
   (footprint "Diode_SMD:D_SOD-123" (layer "B.Cu")
     (at 74.6 84.1 90)
@@
   )
   (footprint "TestPoint:TestPoint_Pad_D1.5mm" (layer "B.Cu")
-    (at 215.85 48.4 180)
+    (at 100.680952 44.2 180)
     (descr "SMD pad as test Point, diameter 1.5mm")
     (tags "test point SMD pad")
@@
   )
   (footprint "TestPoint:TestPoint_Pad_D1.5mm" (layer "B.Cu")
-    (at 225.369048 48.4 180)
+    (at 110.2 44.2 180)
     (descr "SMD pad as test Point, diameter 1.5mm")
     (tags "test point SMD pad")
@@
   (gr_line (start 195.303758 93.981961) (end 195.303758 45.931651) (layer "Edge.Cuts") (width 0.2))
   (gr_circle (center 236.400046 135.930695) (end 237.773608 135.930695) (layer "Edge.Cuts") (width 0.2) (fill none))
-  (gr_line (start 209.695877 42.739423) (end 209.695877 37.359827) (layer "Edge.Cuts") (width 0.2))
+  (gr_line (start 209.695877 32) (end 209.695877 37.359827) (layer "Edge.Cuts") (width 0.2))
   (gr_line (start 155.474869 149.119453) (end 209.377282 149.119453) (layer "Edge.Cuts") (width 0.2))
   (gr_line (start 202.267532 35.489194) (end 193.694947 35.489194) (layer "Edge.Cuts") (width 0.2))
-  (gr_line (start 228.60273 37.359827) (end 228.60273 42.739423) (layer "Edge.Cuts") (width 0.2))
+  (gr_line (start 228.60273 37.359827) (end 228.60273 32) (layer "Edge.Cuts") (width 0.2))
   (gr_arc (start 255.659573 85.106043) (end 255.606555 83.823101) (angle -175.2671709) (layer "Edge.Cuts") (width 0.2))
   (gr_line (start 236.043554 37.359827) (end 228.60273 37.359827) (layer "Edge.Cuts") (width 0.2))
@@
   (gr_line (start 256.471212 147.020908) (end 256.471212 137.726318) (layer "Edge.Cuts") (width 0.2))
   (gr_arc (start 154.003364 147.277263) (end 155.474869 147.163339) (angle -171.1460056) (layer "Edge.Cuts") (width 0.2))
-  (gr_line (start 228.60273 42.739423) (end 209.695877 42.739423) (layer "Edge.Cuts") (width 0.2))
+  (gr_line (start 228.60273 32) (end 209.695877 32) (layer "Edge.Cuts") (width 0.2))
   (gr_arc (start 54.913918 94.675477) (end 54.959219 96.090722) (angle -176.3331845) (layer "Edge.Cuts") (width 0.2))
   (gr_arc (start 54.959219 48.606576) (end 55.171351 50.122276) (angle -164.0656825) (layer "Edge.Cuts") (width 0.2))
