File: RPIZERO/ti92revive.kicad_sch (KiCad schematic)
At the start: 166 parts

Commit message: Clean up and resetting to do the compute modual version
Changed lines of the file:
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@@
     (pin "2")
   )
-  (sheet (at 241.935 80.01) (size 28.575 24.765)
+  (sheet (at 241.935 53.975) (size 28.575 8.89)
     (stroke (width 0.0006) (type solid) (color 0 0 0 0))
     (fill (color 0 0 0 0.0000))
-    (property "Sheet name" "PowerSupply" (id 0) (at 241.935 79.3743 0)
+    (property "Sheet name" "PowerSupply" (id 0) (at 241.935 53.3393 0)
       (effects (font (size 1.27 1.27)) (justify left bottom))
     )
-    (property "Sheet file" "ps.kicad_sch" (id 1) (at 241.935 105.2837 0)
+    (property "Sheet file" "ps.kicad_sch" (id 1) (at 241.935 63.3737 0)
       (effects (font (size 1.27 1.27)) (justify left top))
     )
   )
-  (sheet (at 241.681 22.352) (size 28.448 28.321)
+  (sheet (at 241.681 22.352) (size 28.829 9.398)
     (stroke (width 0.0006) (type solid) (color 0 0 0 0))
     (fill (color 0 0 0 0.0000))
@@
       (effects (font (size 1.27 1.27)) (justify left bottom))
     )
-    (property "Sheet file" "RPICons.kicad_sch" (id 1) (at 241.681 51.1817 0)
+    (property "Sheet file" "RPICons.kicad_sch" (id 1) (at 241.681 32.2587 0)
       (effects (font (size 1.27 1.27)) (justify left top))
     )
   )
-  (sheet (at 241.935 62.484) (size 28.575 8.636)
+  (sheet (at 241.935 38.354) (size 28.575 8.636)
     (stroke (width 0.0006) (type solid) (color 0 0 0 0))
     (fill (color 0 0 0 0.0000))
-    (property "Sheet name" "TestPoints" (id 0) (at 241.935 61.8483 0)
+    (property "Sheet name" "TestPoints" (id 0) (at 241.935 37.7183 0)
       (effects (font (size 1.27 1.27)) (justify left bottom))
     )
-    (property "Sheet file" "TestPoints.kicad_sch" (id 1) (at 241.935 71.6287 0)
+    (property "Sheet file" "TestPoints.kicad_sch" (id 1) (at 241.935 47.4987 0)
       (effects (font (size 1.27 1.27)) (justify left top))
     )
@@
       (reference "#PWR0102") (unit 1) (value "GND") (footprint "")
     )
+    (path "/70488e98-77ad-453e-805e-5550091ec25f/6fb3a625-47b4-4edf-ad0b-23a66b0e7423"
+      (reference "#PWR0108") (unit 1) (value "GND") (footprint "")
+    )
     (path "/70488e98-77ad-453e-805e-5550091ec25f/6f3164af-47a5-484a-9183-9576a35c6557"
       (reference "TP0") (unit 1) (value "GND") (footprint "TestPoint:TestPoint_Pad_D1.5mm")
@@
       (reference "TP4") (unit 1) (value "SDA") (footprint "TestPoint:TestPoint_Pad_D1.5mm")
     )
+    (path "/70488e98-77ad-453e-805e-5550091ec25f/cfe0dbf6-d564-4c70-832a-28734d88d6a9"
+      (reference "TP5") (unit 1) (value "+5v") (footprint "TestPoint:TestPoint_Pad_D1.5mm")
+    )
+    (path "/70488e98-77ad-453e-805e-5550091ec25f/3b8dc35f-e34f-4922-8f56-a330a4248509"
+      (reference "TP6") (unit 1) (value "GND") (footprint "TestPoint:TestPoint_Pad_D1.5mm")
+    )
     (path "/1ac94e0c-d44c-4ee7-9549-80938fb95f34/49de6341-f76e-4ae9-8514-adc2c69f9ef5"
