File: CM4/keypadCons.kicad_sch (KiCad schematic)
At the start: 0 parts

Commit message: Added USB Hub Contoler and usb port internal and external
Parts:
- added C14: CL1, Capacitor_SMD:C_1206_3216Metric, symbol Device:C_Small
- added C15: CL2, Capacitor_SMD:C_1206_3216Metric, symbol Device:C_Small
- added J4, J5: USB_A, Connector_USB:USB_A_Stewart_SS-52100-001_Horizontal, symbol Connector:USB_A
- added R14: 10 M, Resistor_SMD:R_2010_5025Metric_Pad1.40x2.65mm_HandSolder, symbol Device:R_US
- added R15: 9.53K +-1%, Resistor_SMD:R_2010_5025Metric_Pad1.40x2.65mm_HandSolder, symbol Device:R_US
- added R16: 90.9k +-1%, Resistor_SMD:R_2010_5025Metric_Pad1.40x2.65mm_HandSolder, symbol Device:R_US
- added R17: 10k +-1%, Resistor_SMD:R_2010_5025Metric_Pad1.40x2.65mm_HandSolder, symbol Device:R_US
- added TP13: GRSTz, TestPoint:TestPoint_Pad_1.0x1.0mm, symbol Connector:TestPoint
- added TP14: USB_DP_DN4, TestPoint:TestPoint_Pad_1.0x1.0mm, symbol Connector:TestPoint
- added TP15: USB_DM_DN4, TestPoint:TestPoint_Pad_1.0x1.0mm, symbol Connector:TestPoint
- added U7: TUSB4041I, Package_QFP:HTQFP-64-1EP_10x10mm_P0.5mm_EP8x8mm_Mask4.4x4.4mm_ThermalVias, symbol Interface_USB:TUSB4041I
- added Y1: 24 MHz, teensy:HCM49_E, symbol Device:Crystal
Connections:
- new net: C15.1, R14.1, U7.29 (XO), Y1.2
- new net: C14.1, R14.2, U7.30 (XI), Y1.1
- new net: J4.2 (D-), U7.34 (USB_DM_DN1)
- new net: J4.3 (D+), U7.33 (USB_DP_DN1)
- new net: TP14.1, U7.56 (USB_DP_DN4)
- new net: TP15.1, U7.57 (USB_DM_DN4)
- new net: R16.2, R17.1, U7.16 (USB_VBUS)
- new net: J5.2 (D-), U7.42 (USB_DM_DN2)
- new net: J5.3 (D+), U7.41 (USB_DP_DN2)
- new net: TP13.1, U7.18 (GRSTz)
- new net: R15.1, U7.32 (USB_R1)
- new net +5: J4.1 (VBUS), J5.1 (VBUS), R16.1
- new net Earth_Clean: C14.2, C15.2
- new net GND: J4.4 (GND), J4.5 (Shield), J5.4 (GND), J5.5 (Shield), R15.2, R17.2, U7.46 (RSVD)
- new net KEYBOARD_USB_DN: U7.50 (USB_DM_DN3)
- new net KEYBOARD_USB_DP: U7.49 (USB_DP_DN3)
- new net USB_HOST_N: U7.22 (USB_DM_UP)
- new net USB_HOST_P: U7.21 (USB_DP_UP)
