File: CM4/ti92revive.kicad_pcb (KiCad board)
At the start: 2 copper layers, 205 x 116.7 mm, 156 parts, among them J1 USB_B, J2 Conn_01x02, J3 Conn_01x02, J4 USB_A, J5 USB_A, Q1 EMH3, U1 Compute_Module_4_Connectors, U2 NCP114ASN330T1G, U3 BQ25887RGET, U4 MAX17643, U5 ATTINY85-20PU, U6 TQ2SA-L2-3V-Z-Remake, U7 TUSB4041I, Y1 24 MHz

Commit message: Added Keyboard matrix controller and indicator leds
Parts:
- added C16: 10 uF, Capacitor_SMD:C_1206_3216Metric, B.Cu at (97.5, 64.2)
- added C17: 10 uF, Capacitor_SMD:C_1206_3216Metric, B.Cu at (97.5, 70.6)
- added D2: FN, LED_SMD:LED_1206_3216Metric_Pad1.42x1.75mm_HandSolder, F.Cu at (243.6, 38.6)
- added D4: CAPSLOCK, LED_SMD:LED_1206_3216Metric_Pad1.42x1.75mm_HandSolder, F.Cu at (239.9, 38.6)
- added JP2: SolderJumper_2_Open, Jumper:SolderJumper-2_P1.3mm_Open_RoundedPad1.0x1.5mm, B.Cu at (133.8, 118.2)
- added JP3: SolderJumper_2_Open, Jumper:SolderJumper-2_P1.3mm_Open_RoundedPad1.0x1.5mm, B.Cu at (131.2, 118.2)
- added R18: 1K, Resistor_SMD:R_1206_3216Metric, B.Cu at (243.6, 46.4)
- added R20: 1K, Resistor_SMD:R_1206_3216Metric, B.Cu at (238.6, 46.2)
- added TP16: TestPoint, TestPoint:TestPoint_Pad_1.0x1.0mm, B.Cu at (81.8, 74.2)
- added TP17: TestPoint, TestPoint:TestPoint_Pad_1.0x1.0mm, B.Cu at (81.8, 60.2)
- added TP18: TestPoint, TestPoint:TestPoint_Pad_1.0x1.0mm, B.Cu at (81.8, 67.2)
- added TP19: TestPoint, TestPoint:TestPoint_Pad_1.0x1.0mm, B.Cu at (81.8, 53.2)
- added TP20: TestPoint, TestPoint:TestPoint_Pad_1.0x1.0mm, B.Cu at (212.2, 49.2)
- added TP21: TestPoint, TestPoint:TestPoint_Pad_1.0x1.0mm, B.Cu at (215.2, 49.2)
- added TP22: TestPoint, TestPoint:TestPoint_Pad_1.0x1.0mm, B.Cu at (81.8, 81.4)
- added TP23: TestPoint, TestPoint:TestPoint_Pad_1.0x1.0mm, B.Cu at (138.6, 118.2)
- added TP24: TestPoint, TestPoint:TestPoint_Pad_1.0x1.0mm, B.Cu at (127.0, 118.2)
- added U8: TLV740P, Package_TO_SOT_SMD:SOT-23-5_HandSoldering, B.Cu at (97.5, 67.4)
- added U9: SK5126, Package_DFN_QFN:QFN-48-1EP_7x7mm_P0.5mm_EP5.6x5.6mm, B.Cu at (132.2, 125.6)
- C14: value CL1 -> 10pF; moved to B.Cu
- C15: value CL2 -> 10pF; moved to B.Cu
- D1, D81, D82: footprint LED_SMD:LED_2010_5025Metric -> LED_SMD:LED_1206_3216Metric_Pad1.42x1.75mm_HandSolder
- R14, R15, R16, R17, TP13, TP14, TP15, U7, Y1: moved to B.Cu
- moved R17 214.1 mm to (222.8, 112.1), turned to 180 degrees
- moved R16 214.1 mm to (222.8, 107.7), turned to 180 degrees
- moved TP15 209.4 mm to (230.0, 49.2), turned to 180 degrees
- moved TP14 207.3 mm to (227.8, 49.2), turned to 180 degrees
- moved R15 203.8 mm to (222.8, 116.7), turned to 180 degrees
- moved Y1 101.8 mm to (113.9, 78.2), turned to 180 degrees
- moved JP1 100.6 mm to (192.3, 113.4)
- moved Q1 100.6 mm to (185.8, 113.6)
- moved R12 100.6 mm to (185.7, 118.8)
- moved R13 100.6 mm to (185.7, 124.0)
- moved U5 100.6 mm to (198.2, 117.6)
- moved R14 83.4 mm to (116.3, 82.2)
- moved C14 79.8 mm to (117.3, 74.0), turned to 180 degrees
- moved U7 79.7 mm to (113.8, 63.4), turned to 180 degrees
- moved C15 77.8 mm to (110.1, 74.0), turned to 180 degrees
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Connections:
- U7 pad 10: unconnected-(U7-Pad10) -> Net-(U7-Pad10)
- U7 pad 13: unconnected-(U7-Pad13) -> Net-(U7-Pad13)
- U7 pad 19: unconnected-(U7-Pad19) -> +1
- U7 pad 2: unconnected-(U7-Pad2) -> +3.3 High Current
- U7 pad 20: unconnected-(U7-Pad20) -> +3.3 High Current
- U7 pad 25: unconnected-(U7-Pad25) -> +1
- U7 pad 31: unconnected-(U7-Pad31) -> +3.3 High Current
- U7 pad 37: unconnected-(U7-Pad37) -> +1
- U7 pad 45: unconnected-(U7-Pad45) -> +1
- U7 pad 48: unconnected-(U7-Pad48) -> +3.3 High Current
- U7 pad 5: unconnected-(U7-Pad5) -> Net-(U7-Pad5)
- U7 pad 53: unconnected-(U7-Pad53) -> +1
- U7 pad 6: unconnected-(U7-Pad6) -> Net-(U7-Pad6)
- U7 pad 60: unconnected-(U7-Pad60) -> +1
- U7 pad 63: unconnected-(U7-Pad63) -> +1
- U7 pad 65: unconnected-(U7-Pad65) -> GND
- U7 pad 7: unconnected-(U7-Pad7) -> Net-(U7-Pad7)
- U7 pad 8: unconnected-(U7-Pad8) -> Net-(U7-Pad8)
- U7 pad 9: unconnected-(U7-Pad9) -> Net-(U7-Pad9)
Other:
- board text removed: "Not in final Position"
