File: CM4/_autosave-ps.kicad_sch (KiCad schematic)
At the start: 48 parts, among them J1 USB_B, J2 Bat0, J3 Bat1, Q1 EMH3, U2 NCP114ASN330T1G, U3 BQ25887RGET, U4 MAX17643, U5 ATTINY85-20PU, U6 TQ2SA-L2-3V-Z-Remake, U8 TLV740P

Commit message: 100 things left to rout
Parts:
- added TP25: TestPoint, TestPoint:TestPoint_Pad_D1.0mm, symbol Connector:TestPoint
Connections:
- net at U5.1 (PB5): now also TP25.1
