File: CM4/ti92revive.kicad_sch (KiCad schematic)
At the start: 84 parts

Commit message: Finally Added the display!!!!
Other:
- added sheet DisplayStuff (display.kicad_sch)
Changed lines of the file:
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@@
     (pin "2")
+  )
+  (sheet (at 241.935 85.725) (size 28.575 10.16)
+    (stroke (width 0.0006) (type solid) (color 0 0 0 0))
+    (fill (color 0 0 0 0.0000))
+    (property "Sheet name" "DisplayStuff" (id 0) (at 241.935 85.0893 0)
+      (effects (font (size 1.27 1.27)) (justify left bottom))
+    )
+    (property "Sheet file" "display.kicad_sch" (id 1) (at 241.935 96.3937 0)
+      (effects (font (size 1.27 1.27)) (justify left top))
+    )
   )
   (sheet (at 241.935 53.975) (size 28.575 8.89)
@@
     (path "/1ac94e0c-d44c-4ee7-9549-80938fb95f34/" (page "4"))
     (path "/60beade3-25b6-4075-b5fd-5a6340fab42e/" (page "5"))
+    (path "/deaa2a42-5edf-49d0-a8e0-8ad38d123749/" (page "6"))
   )
   (symbol_instances
@@
       (reference "Y1") (unit 1) (value "24 MHz") (footprint "teensy:HCM49_E")
     )
+    (path "/deaa2a42-5edf-49d0-a8e0-8ad38d123749/0a2dc4dd-32ec-4063-981a-f996d8e100db"
+      (reference "#PWR0148") (unit 1) (value "GND") (footprint "")
+    )
+    (path "/deaa2a42-5edf-49d0-a8e0-8ad38d123749/17af90c7-cb82-4fb1-a7ed-762b203b4f09"
+      (reference "U10") (unit 1) (value "4inch_RPi_LCD_(C)") (footprint "Connector_PinSocket_2.54mm:PinSocket_2x13_P2.54mm_Vertical")
+    )
   )

Commit message: Started the "fun" of routing
Parts:
- arrwDWN1, arrwLeft1, arrwRight1, arrwUP1, kb2nd1, kbA1, kbALT1, kbALTG1, kbAPPS1, kbB1, kbBKSP1, kbC1, kbCOS1, kbClear1, kbComa1, kbD1, kbDiv1, kbDot1, kbDot2, kbENT1, kbESC1, kbESC55, kbF1, kbG1, kbH1, kbI1, kbJ1, kbK1, kbL1, kbLBrack1, kbLn1, kbM1, kbMode1, kbMult1, kbN1, kbN2, kbN3, kbN4, kbN5, kbN6, kbN8, kbO1, kbP1, kbPI1, kbPLUS1, kbQ1, kbR1, kbRBrack1, kbRET1, kbRET32, kbS1, kbSIN1, kbShiftL1, kbSpace1, kbSpace2, kbT1, kbTAB1, kbU1, kbV1, kbW1, kbX1, kbY1, kbZ1, kf4, kf5, kf6, kf7, kf8, kwE1: footprint Button_Switch_SMD:SW_SPST_B3SL-1002P -> lib:Kbpad
- kN666, kbAPPS2, kbAnex2, kbEnterNum1, kbEnterNum66, kbMinus1, kbN521, kbN7, kbN9, kbNeg1, kbTAN1, kf1, kf2, kf3, klock1: footprint 18650:Kbpad -> lib:Kbpad
Connections:
- net col1: no longer arrwLeft1.1, kbA1.2, kbALT1.1, kbALTG1.1, kbAPPS1.1, kbAPPS2.1, kbB1.1, kbB1.2, kbBKSP1.2, kbC1.1, kbC1.2, kbClear1.1, kbComa1.1, kbD1.1, kbD1.2, kbDiv1.1, kbDot1.1, kbDot2.2, kbEnterNum1.1, kbEnterNum66.1, kbF1.1, kbF1.2, kbG1.1, kbG1.2, kbH1.1, kbH1.2, kbI1.2, kbJ1.1, kbJ1.2, kbK1.2, kbL1.2, kbLn1.1, kbM1.2, kbMode1.1, kbN3.1, kbN4.1, kbN5.1, kbN521.1, kbN6.1, kbN6.2, kbN7.1, kbNeg1.1, kbO1.2, kbP1.2, kbPLUS1.1, kbQ1.2, kbR1.1, kbR1.2, kbRBrack1.1, kbRET1.2, kbRET32.2, kbS1.2, kbSpace1.1, kbSpace2.1, kbT1.1, kbT1.2, kbTAB1.2, kbU1.1, kbU1.2, kbV1.1, kbV1.2, kbW1.2, kbX1.1, kbX1.2, kbY1.1, kbY1.2, kbZ1.2, kf2.1, kf3.1, kf4.1, kf5.1, kf6.1, kwE1.1, kwE1.2
- new net col2: kbALT1.1, kbD1.1, kbMode1.1, kbN3.1, kbRBrack1.1, kbX1.1, kf2.1, kwE1.1
- new net col3: kbC1.1, kbClear1.1, kbComa1.1, kbF1.1, kbPLUS1.1, kbR1.1, kbSpace1.1, kbSpace2.1, kf3.1
- new net col4: kbALTG1.1, kbDiv1.1, kbG1.1, kbLn1.1, kbN4.1, kbT1.1, kbV1.1, kf4.1
- new net col5: kbA1.2, kbAPPS1.1, kbAPPS2.1, kbB1.1, kbBKSP1.2, kbD1.2, kbDot1.1, kbF1.2, kbG1.2, kbH1.1, kbH1.2, kbJ1.2, kbK1.2, kbL1.2, kbN5.1, kbN521.1, kbS1.2, kbY1.1, kf5.1
- new net col6: arrwLeft1.1, kbEnterNum1.1, kbEnterNum66.1, kbJ1.1, kbN6.1, kbN7.1, kbNeg1.1, kbU1.1, kf6.1
- new net row1: kbI1.2, kbO1.2, kbP1.2, kbQ1.2, kbR1.2, kbT1.2, kbU1.2, kbW1.2, kbY1.2, kwE1.2
- new net row3: kbB1.2, kbC1.2, kbDot2.2, kbM1.2, kbN6.2, kbRET1.2, kbRET32.2, kbTAB1.2, kbV1.2, kbX1.2, kbZ1.2
Other:
- moved on the sheet: kbD1, kbF1, kbG1, kbH1, kbJ1, kbS1, kbSpace1, kbSpace2

Commit message: i hate routing
Connections:
- net col5: no longer kbA1.2, kbBKSP1.2, kbD1.2, kbF1.2, kbG1.2, kbH1.2, kbJ1.2, kbK1.2, kbL1.2, kbS1.2
- new net row2: kbA1.2, kbBKSP1.2, kbD1.2, kbF1.2, kbG1.2, kbH1.2, kbJ1.2, kbK1.2, kbL1.2, kbS1.2
Changed lines of the file:
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@@
   (junction (at 147.32 45.72) (diameter 1.016) (color 0 0 0 0))
   (junction (at 147.32 57.785) (diameter 1.016) (color 0 0 0 0))
-  (junction (at 147.32 66.04) (diameter 1.016) (color 0 0 0 0))
   (junction (at 147.32 68.58) (diameter 1.016) (color 0 0 0 0))
   (junction (at 147.32 81.28) (diameter 1.016) (color 0 0 0 0))
@@
     (stroke (width 0) (type solid) (color 0 0 0 0))
   )
-  (wire (pts (xy 134.62 66.04) (xy 147.32 66.04))
+  (wire (pts (xy 134.62 66.04) (xy 152.4 66.04))
     (stroke (width 0) (type solid) (color 0 0 0 0))
   )
@@
     (stroke (width 0) (type solid) (color 0 0 0 0))
   )
-  (wire (pts (xy 147.32 57.785) (xy 147.32 66.04))
-    (stroke (width 0) (type solid) (color 0 0 0 0))
-  )
-  (wire (pts (xy 147.32 66.04) (xy 147.32 68.58))
-    (stroke (width 0) (type solid) (color 0 0 0 0))
-  )
-  (wire (pts (xy 147.32 66.04) (xy 152.4 66.04))
-    (stroke (width 0) (type solid) (color 0 0 0 0))
-  )
+  (wire (pts (xy 147.32 57.785) (xy 147.32 68.58))
+    (stroke (width 0) (type solid) (color 0 0 0 0))
+  )
