File: CM4/ti92revive.kicad_sch (KiCad schematic)
At the start: 84 parts

Commit message: Bigone here we go
Whats gonna happon is im gonna get a 4 inch hdmi display and desolder the hdmi connector and add it to a ribbion cable and then add a connector to the pcb for hdmi to interface with that
Other:
- note added: "TODO: Add SDCARD Slot Display"
Changed lines of the file:
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@@
     (effects (font (size 1.524 1.524)) (justify left bottom))
+  )
+  (text "TODO:\nAdd SDCARD Slot\nDisplay " (at 68.58 144.145 180)
+    (effects (font (size 1.27 1.27)) (justify right bottom))
   )
   (label "row0" (at 30.48 43.18 0)
@@
       (reference "Y1") (unit 1) (value "24 MHz") (footprint "teensy:HCM49_E")
     )
-    (path "/deaa2a42-5edf-49d0-a8e0-8ad38d123749/0a2dc4dd-32ec-4063-981a-f996d8e100db"
-      (reference "#PWR0148") (unit 1) (value "GND") (footprint "")
-    )
-    (path "/deaa2a42-5edf-49d0-a8e0-8ad38d123749/9518133d-6049-47a4-86a3-4d24f6fa40a6"
-      (reference "#PWR0149") (unit 1) (value "GND") (footprint "")
-    )
-    (path "/deaa2a42-5edf-49d0-a8e0-8ad38d123749/80f757e9-897b-4aed-8a1e-6dc617685752"
-      (reference "#PWR0150") (unit 1) (value "GND") (footprint "")
-    )
-    (path "/deaa2a42-5edf-49d0-a8e0-8ad38d123749/e8d94436-431a-4be0-80a1-acacd5ee34da"
-      (reference "#PWR0151") (unit 1) (value "GND") (footprint "")
-    )
-    (path "/deaa2a42-5edf-49d0-a8e0-8ad38d123749/f7bd4909-5231-41d0-bb21-aca3b104a336"
-      (reference "#PWR0152") (unit 1) (value "GND") (footprint "")
-    )
-    (path "/deaa2a42-5edf-49d0-a8e0-8ad38d123749/72ed022f-9aa1-42af-931c-46ec3d0422a6"
-      (reference "U10") (unit 1) (value "4inch_RPi_LCD_(C)") (footprint "")
-    )
-  )
+    (path "/deaa2a42-5edf-49d0-a8e0-8ad38d123749/202ac646-4d90-48da-b41b-80fce3ff1bfd"
+      (reference "J?") (unit 1) (value "HDMI_A_1.4") (footprint "")
+    )
+  )

Commit message: added sdcard
Other:
- added sheet SDCard (SDCard.kicad_sch)
Changed lines of the file:
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@@
+    )
+  )
+  (sheet (at 241.935 104.775) (size 28.575 13.335)
+    (stroke (width 0.0006) (type solid) (color 0 0 0 0))
+    (fill (color 0 0 0 0.0000))
+    (property "Sheet name" "SDCard" (id 0) (at 241.935 104.1393 0)
+      (effects (font (size 1.27 1.27)) (justify left bottom))
+    )
+    (property "Sheet file" "SDCard.kicad_sch" (id 1) (at 241.935 118.6187 0)
+      (effects (font (size 1.27 1.27)) (justify left top))
     )
   )
@@
     (path "/60beade3-25b6-4075-b5fd-5a6340fab42e/" (page "5"))
     (path "/deaa2a42-5edf-49d0-a8e0-8ad38d123749/" (page "6"))
+    (path "/3967c5d9-7139-462e-85dd-613180c27708/" (page "7"))
   )
   (symbol_instances
@@
       (reference "J6") (unit 1) (value "ZF5S-20-01-T-WT") (footprint "SAMTEC_ZF5S-20-01-T-WT")
     )
+    (path "/3967c5d9-7139-462e-85dd-613180c27708/46b93ecf-e78c-48e7-a0cb-c8181f7860a1"
+      (reference "#PWR?") (unit 1) (value "GND") (footprint "")
+    )
+    (path "/3967c5d9-7139-462e-85dd-613180c27708/f5a17727-f806-48c2-9ce9-0b13d097a625"
+      (reference "#PWR?") (unit 1) (value "GND") (footprint "")
+    )
+    (path "/3967c5d9-7139-462e-85dd-613180c27708/b6337edd-4f17-42f1-b0a2-dcc794480dbc"
+      (reference "C?") (unit 1) (value "10 uF") (footprint "Capacitor_SMD:C_1206_3216Metric")
+    )
+    (path "/3967c5d9-7139-462e-85dd-613180c27708/0c265a58-dc9d-41fb-b30b-f67b537f5fdd"
+      (reference "J?") (unit 1) (value "Micro_SD_Card") (footprint "")
+    )
   )

Commit message: display done
Other:
- note added: "TODO: Backlight Power Control"
- note removed: "TODO: Add SDCARD Slot Display"
Changed lines of the file:
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@@
     (effects (font (size 1.524 1.524)) (justify left bottom))
   )
-  (text "TODO:\nAdd SDCARD Slot\nDisplay " (at 68.58 144.145 180)
+  (text "TODO:\nBacklight Power Control\n" (at 90.805 156.845 180)
     (effects (font (size 1.27 1.27)) (justify right bottom))
   )
@@
       (reference "J6") (unit 1) (value "ZF5S-20-01-T-WT") (footprint "SAMTEC_ZF5S-20-01-T-WT")
     )
+    (path "/3967c5d9-7139-462e-85dd-613180c27708/f5a17727-f806-48c2-9ce9-0b13d097a625"
+      (reference "#PWR0148") (unit 1) (value "GND") (footprint "")
+    )
     (path "/3967c5d9-7139-462e-85dd-613180c27708/46b93ecf-e78c-48e7-a0cb-c8181f7860a1"
-      (reference "#PWR?") (unit 1) (value "GND") (footprint "")
-    )
-    (path "/3967c5d9-7139-462e-85dd-613180c27708/f5a17727-f806-48c2-9ce9-0b13d097a625"
-      (reference "#PWR?") (unit 1) (value "GND") (footprint "")
+      (reference "#PWR0149") (unit 1) (value "GND") (footprint "")
     )
     (path "/3967c5d9-7139-462e-85dd-613180c27708/b6337edd-4f17-42f1-b0a2-dcc794480dbc"
-      (reference "C?") (unit 1) (value "10 uF") (footprint "Capacitor_SMD:C_1206_3216Metric")
+      (reference "C18") (unit 1) (value "10 uF") (footprint "Capacitor_SMD:C_1206_3216Metric")
     )
     (path "/3967c5d9-7139-462e-85dd-613180c27708/0c265a58-dc9d-41fb-b30b-f67b537f5fdd"
-      (reference "J?") (unit 1) (value "Micro_SD_Card") (footprint "")
-    )
-  )
+      (reference "J7") (unit 1) (value "Micro_SD_Card") (footprint "teensy:MOLEX_503182-1852")
+    )
+  )

Commit message: Compleated REV001
Other:
- note removed: "TODO: Backlight Power Control"
Changed lines of the file:
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@@
     (effects (font (size 1.524 1.524)) (justify left bottom))
-  )
-  (text "TODO:\nBacklight Power Control\n" (at 90.805 156.845 180)
-    (effects (font (size 1.27 1.27)) (justify right bottom))
   )
   (label "row0" (at 30.48 43.18 0)
@@
       (reference "Y1") (unit 1) (value "24 MHz") (footprint "teensy:HCM49_E")
     )
+    (path "/deaa2a42-5edf-49d0-a8e0-8ad38d123749/27ce00c4-639c-4961-84ff-2278e1a07cf5"
+      (reference "#PWR0150") (unit 1) (value "GND") (footprint "")
+    )
     (path "/deaa2a42-5edf-49d0-a8e0-8ad38d123749/f3ed8bb6-6f6d-45b9-a57c-809a63eabf0d"
       (reference "#PWR0152") (unit 1) (value "GND") (footprint "")
@@
       (reference "J6") (unit 1) (value "ZF5S-20-01-T-WT") (footprint "SAMTEC_ZF5S-20-01-T-WT")
     )
+    (path "/deaa2a42-5edf-49d0-a8e0-8ad38d123749/273ad236-dd19-447e-87f6-31e2d897e56e"
+      (reference "J8") (unit 1) (value "Conn_01x02_Male") (footprint "Connector_PinHeader_1.00mm:PinHeader_1x02_P1.00mm_Vertical")
+    )
     (path "/3967c5d9-7139-462e-85dd-613180c27708/f5a17727-f806-48c2-9ce9-0b13d097a625"
