File: CM4/TestPoints.kicad_sch (KiCad schematic)
At the start: 10 parts

Commit message: Adding image for readme
Parts:
- removed TP8: 14, TestPoint:TestPoint_Pad_D1.5mm, symbol Connector:TestPoint
- removed TP9: 15, TestPoint:TestPoint_Pad_D1.5mm, symbol Connector:TestPoint
Changed lines of the file:
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@@
-    )
-  )
-  (global_label "SerialPin14" (shape input) (at 106.68 133.35 270)
-    (effects (font (size 1.27 1.27)) (justify right))
-    (property "Intersheet References" "${INTERSHEET_REFS}" (id 0) (at 106.6006 146.7093 90)
-      (effects (font (size 1.27 1.27)) (justify right) hide)
-    )
-  )
-  (global_label "SerialPin15" (shape input) (at 116.205 133.35 270)
-    (effects (font (size 1.27 1.27)) (justify right))
-    (property "Intersheet References" "${INTERSHEET_REFS}" (id 0) (at 116.1256 146.7093 90)
-      (effects (font (size 1.27 1.27)) (justify right) hide)
     )
   )
@@
       (effects (font (size 1.27 1.27)) hide)
     )
-    (pin "1")
-  )
-  (symbol (lib_id "Connector:TestPoint") (at 106.68 133.35 0) (unit 1)
-    (in_bom yes) (on_board yes)
-    (property "Reference" "TP8" (id 0) (at 108.0771 130.7476 0)
-      (effects (font (size 1.27 1.27)) (justify left))
-    )
-    (property "Value" "14" (id 1) (at 108.0771 133.0463 0)
-      (effects (font (size 1.27 1.27)) (justify left))
-    )
-    (property "Footprint" "TestPoint:TestPoint_Pad_D1.5mm" (id 2) (at 111.76 133.35 0)
-      (effects (font (size 1.27 1.27)) hide)
-    )
-    (property "Datasheet" "~" (id 3) (at 111.76 133.35 0)
-      (effects (font (size 1.27 1.27)) hide)
-    )
-    (pin "1")
-  )
-  (symbol (lib_id "Connector:TestPoint") (at 116.205 133.35 0) (unit 1)
-    (in_bom yes) (on_board yes)
-    (property "Reference" "TP9" (id 0) (at 117.6021 130.7476 0)
-      (effects (font (size 1.27 1.27)) (justify left))
-    )
-    (property "Value" "15" (id 1) (at 117.6021 133.0463 0)
-      (effects (font (size 1.27 1.27)) (justify left))
-    )
-    (property "Footprint" "TestPoint:TestPoint_Pad_D1.5mm" (id 2) (at 121.285 133.35 0)
-      (effects (font (size 1.27 1.27)) hide)
-    )
-    (property "Datasheet" "~" (id 3) (at 121.285 133.35 0)
-      (effects (font (size 1.27 1.27)) hide)
-    )

Commit message: PrepedHDMIConnections
Parts:
- added TP26: GND, TestPoint:TestPoint_Pad_D1.5mm, symbol Connector:TestPoint
- added TP8: SP14, TestPoint:TestPoint_Pad_D1.5mm, symbol Connector:TestPoint
- added TP9: SP15, TestPoint:TestPoint_Pad_D1.5mm, symbol Connector:TestPoint
Connections:
- net GND: now also TP26.1
- new net SerialPin14: TP8.1
- new net SerialPin15: TP9.1
Other:
- moved on the sheet: TP7
Changed lines of the file:
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@@
+    )
+  )
+  (global_label "SerialPin14" (shape input) (at 189.23 114.3 270)
+    (effects (font (size 1.27 1.27)) (justify right))
+    (property "Intersheet References" "${INTERSHEET_REFS}" (id 0) (at 189.1506 127.6593 90)
+      (effects (font (size 1.27 1.27)) (justify right) hide)
+    )
+  )
+  (global_label "SerialPin15" (shape input) (at 196.85 114.3 270)
+    (effects (font (size 1.27 1.27)) (justify right))
+    (property "Intersheet References" "${INTERSHEET_REFS}" (id 0) (at 196.7706 127.6593 90)
+      (effects (font (size 1.27 1.27)) (justify right) hide)
     )
   )
@@
     (pin "1")
   )
-  (symbol (lib_id "Connector:TestPoint") (at 97.155 133.35 0) (unit 1)
-    (in_bom yes) (on_board yes)
-    (property "Reference" "TP7" (id 0) (at 98.5521 130.7476 0)
-      (effects (font (size 1.27 1.27)) (justify left))
-    )
-    (property "Value" "GND" (id 1) (at 98.5521 133.0463 0)
-      (effects (font (size 1.27 1.27)) (justify left))
-    )
-    (property "Footprint" "TestPoint:TestPoint_Pad_D1.5mm" (id 2) (at 102.235 133.35 0)
-      (effects (font (size 1.27 1.27)) hide)
-    )
-    (property "Datasheet" "~" (id 3) (at 102.235 133.35 0)
-      (effects (font (size 1.27 1.27)) hide)
-    )
-    (pin "1")
-  )
   (symbol (lib_id "Connector:TestPoint") (at 106.045 114.3 0) (unit 1)
     (in_bom yes) (on_board yes)
@@
     )
     (property "Datasheet" "~" (id 3) (at 173.99 114.3 0)
+      (effects (font (size 1.27 1.27)) hide)
+    )
+    (pin "1")
+  )
+  (symbol (lib_id "Connector:TestPoint") (at 189.23 114.3 0) (unit 1)
+    (in_bom yes) (on_board yes)
+    (property "Reference" "TP8" (id 0) (at 190.6271 111.6976 0)
+      (effects (font (size 1.27 1.27)) (justify left))
+    )
+    (property "Value" "SP14" (id 1) (at 190.6271 113.9963 0)
+      (effects (font (size 1.27 1.27)) (justify left))
+    )
+    (property "Footprint" "TestPoint:TestPoint_Pad_D1.5mm" (id 2) (at 194.31 114.3 0)
+      (effects (font (size 1.27 1.27)) hide)
+    )
+    (property "Datasheet" "~" (id 3) (at 194.31 114.3 0)
+      (effects (font (size 1.27 1.27)) hide)
+    )
+    (pin "1")
+  )
+  (symbol (lib_id "Connector:TestPoint") (at 196.85 114.3 0) (unit 1)
+    (in_bom yes) (on_board yes)
+    (property "Reference" "TP9" (id 0) (at 198.2471 111.6976 0)
+      (effects (font (size 1.27 1.27)) (justify left))
+    )
+    (property "Value" "SP15" (id 1) (at 198.2471 113.9963 0)
+      (effects (font (size 1.27 1.27)) (justify left))
+    )
+    (property "Footprint" "TestPoint:TestPoint_Pad_D1.5mm" (id 2) (at 201.93 114.3 0)
+      (effects (font (size 1.27 1.27)) hide)
+    )
+    (property "Datasheet" "~" (id 3) (at 201.93 114.3 0)
+      (effects (font (size 1.27 1.27)) hide)
+    )
+    (pin "1")
+  )
+  (symbol (lib_id "Connector:TestPoint") (at 206.375 114.3 0) (unit 1)
+    (in_bom yes) (on_board yes)
+    (property "Reference" "TP7" (id 0) (at 207.7721 111.6976 0)
+      (effects (font (size 1.27 1.27)) (justify left))
+    )
+    (property "Value" "GND" (id 1) (at 207.7721 113.9963 0)
+      (effects (font (size 1.27 1.27)) (justify left))
+    )
+    (property "Footprint" "TestPoint:TestPoint_Pad_D1.5mm" (id 2) (at 211.455 114.3 0)
+      (effects (font (size 1.27 1.27)) hide)
+    )
+    (property "Datasheet" "~" (id 3) (at 211.455 114.3 0)
+      (effects (font (size 1.27 1.27)) hide)
+    )
+    (pin "1")
+  )
+  (symbol (lib_id "Connector:TestPoint") (at 213.36 114.3 0) (unit 1)
+    (in_bom yes) (on_board yes)
+    (property "Reference" "TP26" (id 0) (at 214.7571 111.6976 0)
+      (effects (font (size 1.27 1.27)) (justify left))
+    )
+    (property "Value" "GND" (id 1) (at 214.7571 113.9963 0)
+      (effects (font (size 1.27 1.27)) (justify left))
+    )
+    (property "Footprint" "TestPoint:TestPoint_Pad_D1.5mm" (id 2) (at 218.44 114.3 0)
+      (effects (font (size 1.27 1.27)) hide)
+    )
+    (property "Datasheet" "~" (id 3) (at 218.44 114.3 0)
       (effects (font (size 1.27 1.27)) hide)
     )
@@
     (pin "1")
   )
-  (symbol (lib_id "power:GND") (at 97.155 133.35 0) (unit 1)
-    (in_bom yes) (on_board yes)
-    (property "Reference" "#PWR0111" (id 0) (at 97.155 139.7 0)
-      (effects (font (size 1.27 1.27)) hide)
-    )
-    (property "Value" "GND" (id 1) (at 97.155 137.6744 0))
-    (property "Footprint" "" (id 2) (at 97.155 133.35 0)
-      (effects (font (size 1.27 1.27)) hide)
-    )
-    (property "Datasheet" "" (id 3) (at 97.155 133.35 0)
-      (effects (font (size 1.27 1.27)) hide)
-    )
-    (pin "1")
-  )
   (symbol (lib_id "power:GND") (at 123.19 114.3 0) (unit 1)
     (in_bom yes) (on_board yes)
@@
       (effects (font (size 1.27 1.27)) hide)
     )
+    (pin "1")
+  )
+  (symbol (lib_id "power:GND") (at 206.375 114.3 0) (unit 1)
+    (in_bom yes) (on_board yes)
+    (property "Reference" "#PWR0111" (id 0) (at 206.375 120.65 0)
+      (effects (font (size 1.27 1.27)) hide)
+    )
+    (property "Value" "GND" (id 1) (at 206.375 118.6244 0))
+    (property "Footprint" "" (id 2) (at 206.375 114.3 0)
+      (effects (font (size 1.27 1.27)) hide)
+    )
+    (property "Datasheet" "" (id 3) (at 206.375 114.3 0)
+      (effects (font (size 1.27 1.27)) hide)
+    )
+    (pin "1")
+  )
+  (symbol (lib_id "power:GND") (at 213.36 114.3 0) (unit 1)
+    (in_bom yes) (on_board yes)
+    (property "Reference" "#PWR0153" (id 0) (at 213.36 120.65 0)
+      (effects (font (size 1.27 1.27)) hide)
+    )
+    (property "Value" "GND" (id 1) (at 213.36 118.6244 0))
+    (property "Footprint" "" (id 2) (at 213.36 114.3 0)
+      (effects (font (size 1.27 1.27)) hide)
+    )
+    (property "Datasheet" "" (id 3) (at 213.36 114.3 0)
+      (effects (font (size 1.27 1.27)) hide)
+    )
