File: CM4/SDCard.kicad_sch (KiCad schematic)
At the start: 2 parts

Commit message: display done
Parts:
- J7: renamed from J?; footprint (none) -> teensy:MOLEX_503182-1852
- gave numbers to parts that had none: 1
Changed lines of the file:
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@@
   (symbol (lib_id "power:GND") (at 163.83 106.68 0) (unit 1)
     (in_bom yes) (on_board yes)
-    (property "Reference" "#PWR?" (id 0) (at 163.83 113.03 0)
+    (property "Reference" "#PWR0148" (id 0) (at 163.83 113.03 0)
       (effects (font (size 1.27 1.27)) hide)
     )
@@
   (symbol (lib_id "power:GND") (at 226.695 116.84 0) (unit 1)
     (in_bom yes) (on_board yes)
-    (property "Reference" "#PWR?" (id 0) (at 226.695 123.19 0)
+    (property "Reference" "#PWR0149" (id 0) (at 226.695 123.19 0)
       (effects (font (size 1.27 1.27)) hide)
     )
@@
   (symbol (lib_id "Device:C_Small") (at 163.83 104.14 0) (unit 1)
     (in_bom yes) (on_board yes)
-    (property "Reference" "C?" (id 0) (at 155.9942 102.7441 0)
+    (property "Reference" "C18" (id 0) (at 155.9942 102.7441 0)
       (effects (font (size 1.27 1.27)) (justify left))
     )
@@
   (symbol (lib_id "Connector:Micro_SD_Card") (at 206.375 101.6 0) (unit 1)
     (in_bom yes) (on_board yes)
-    (property "Reference" "J?" (id 0) (at 205.105 84.1968 0))
+    (property "Reference" "J7" (id 0) (at 205.105 84.1968 0))
     (property "Value" "Micro_SD_Card" (id 1) (at 205.105 86.4955 0))
-    (property "Footprint" "" (id 2) (at 235.585 93.98 0)
+    (property "Footprint" "teensy:MOLEX_503182-1852" (id 2) (at 235.585 93.98 0)
       (effects (font (size 1.27 1.27)) hide)
     )
